Commit message: Figured out how to do srdf

File: switch-flipper/src/arm_control/config/urdf/wx200-ee.urdf.xacro (robot description, xacro)
@@ -6,4 +6,6 @@
     <xacro:property name="arm_tag_mount_mesh" value="package://arm_control/meshes/arm_april_tag.stl"/>
     <joint name="lollypop_joint" type="fixed">
+                <!-- Interbotix have axis for all fixed joint.-->
+                <axis xyz="1 0 0"/>
         <origin xyz="0.0 0.0 0.0" rpy="0.0 0.0 0.0"/>
         <parent link="$(arg robot_name)/fingers_link"/>
@@ -32,4 +34,24 @@
         </collision>
     </link>
+    <joint name="lollypop_ee_offset" type="fixed">
+        <!-- Interbotix have axis for all fixed joint.-->
+        <axis xyz="1 0 0"/>
+        <origin xyz="0.055 0.0 0.0" rpy="0.0 0.0 0.0"/>
+        <parent link="lollypop_hammer"/>
+        <child link="lollypop_ee_link"/>
+    </joint>
+    <link name="lollypop_ee_link">
+    <inertial>
+        <mass value="0.001"/>
+        <inertia
+          ixx="0.001"
+          iyy="0.001"
+          izz="0.001"
+          ixy="0"
+          ixz="0"
+          iyz="0"/>
+      </inertial>
+    </link>
+    <!-- All joints and links related to camera -->
     <joint name="camera_stand_joint" type="fixed">
         <origin xyz="0.0 0.0 0.0" rpy="0.0 0.0 0.0"/>
@@ -66,4 +88,5 @@
     </joint>
     <link name="camera_mount"/>
+    <!-- All joints and links related to apriltag -->
     <joint name="april_tag_mount_joint" type="fixed">
         <origin xyz="0.0 0.0 0.0" rpy="0.0 0.0 0.0"/>
