Commit message: Create a split on wx200 URDF, so locobot could find a simple version to use.

File: switch-flipper/src/arm_control/config/srdf/wx200-ee-fixedcamera.srdf.xacro (robot description, xacro)
@@ -19,4 +19,16 @@
     <!-- and between finger and april tag mount -->
     <disable_collisions link1="lollypop_hammer" link2="april_tag_mount" reason="Never" />
+    <!-- April tag mount also need to be ignored between all the finger related stuff. same as above  -->
+    <disable_collisions link1="april_tag_mount" link2="$(arg robot_name)/gripper_bar_link" reason="Adjacent" />
+    <disable_collisions link1="april_tag_mount" link2="$(arg robot_name)/left_finger_link" reason="Adjacent" />
+    <disable_collisions link1="april_tag_mount" link2="$(arg robot_name)/right_finger_link" reason="Adjacent" />
+    <disable_collisions link1="april_tag_mount" link2="$(arg robot_name)/gripper_prop_link" reason="Never" />
+    <disable_collisions link1="april_tag_mount" link2="$(arg robot_name)/gripper_link" reason="Never" />
+    <disable_collisions link1="april_tag_mount" link2="$(arg robot_name)/wrist_link" reason="Never" />
+    <!-- Also all forearm link , because the joint limit doesn't allow collision anyway.  -->
+    <disable_collisions link1="april_tag_mount" link2="$(arg robot_name)/forearm_link" reason="Never" />
+    <!-- The camera mount won't collide with base and two showder motor -->
+    <disable_collisions link1="camera_stand" link2="$(arg robot_name)/base_link" reason="Adjacent" />
+    <disable_collisions link1="camera_stand" link2="$(arg robot_name)/shoulder_link" reason="Never" />
     <group name="lollypop_hammer">
         <joint name="waist" />

File: switch-flipper/src/arm_control/config/urdf/wx200-ee.urdf.xacro (robot description, xacro)
@@ -53,73 +53,3 @@
       </inertial>
     </link>
-    <!-- All joints and links related to camera -->
-    <joint name="camera_stand_joint" type="fixed">
-        <origin xyz="0.0 0.0 0.0" rpy="0.0 0.0 0.0"/>
-        <parent link="$(arg robot_name)/base_link"/>
-        <child link="camera_stand"/>
-    </joint>
-    <link name="camera_stand">
-        <inertial>
-            <origin xyz="0.0 0.0 0.0" rpy="0.0 0.0 0.0"/>
-            <mass value="0.001"/>
-            <inertia ixx="0.0" ixy="0.0" ixz="0.0" iyy="0.0" iyz="0.0" izz="0.0"/>
-        </inertial>
-        <visual name="">
-            <origin xyz="0.0 0.0 0.0" rpy="0.0 0.0 0.0"/>
-            <geometry>
-                <mesh filename="${camera_stand_mesh}" scale="1.0 1.0 1.0"/>
-            </geometry>
-            <material name="">
-                <color rgba="1.0 0.0 0.0 0.95"/>
-            </material>
-        </visual>
-        <collision>
-            <origin xyz="0.0 0.0 0.0" rpy="0.0 0.0 0.0"/>
-            <geometry>
-                <mesh filename="${camera_stand_mesh}" scale="1.0 1.0 1.0"/>
-            </geometry>
-        </collision>
-    </link>
-    <joint name="to_camer_mount_offset" type="fixed">
-        <!-- The X offset decide on which mounting point it is using, -60mm for the rare one -->
-        <origin xyz="-0.060 -0.1765 0.143" rpy="0.0 0.0 0.0"/>
-        <parent link="camera_stand"/>
-        <child link="camera_mount"/>
-    </joint>
-    <link name="camera_mount"/>
-    <!-- All joints and links related to apriltag -->
-    <joint name="april_tag_mount_joint" type="fixed">
-        <origin xyz="0.0 0.0 0.0" rpy="0.0 0.0 0.0"/>
-        <parent link="$(arg robot_name)/fingers_link"/>
-        <child link="april_tag_mount"/>
-    </joint>
-    <link name="april_tag_mount">
-        <inertial>
-            <!-- These are onshape output value. -->
-            <origin xyz="-16.6 0.0 30.6" rpy="0.0 0.0 0.0"/>
-            <mass value="0.03"/>
-            <inertia ixx="0.093" ixy="0.0" ixz="0.005" iyy="0.03" iyz="0.0" izz="0.112"/>
-        </inertial>
-        <visual name="">
-            <origin xyz="0.0 0.0 0.0" rpy="0.0 0.0 0.0"/>
-            <geometry>
-                <mesh filename="${arm_tag_mount_mesh}" scale="1.0 1.0 1.0"/>
-            </geometry>
-            <material name="">
-                <color rgba="0.85 0.70 1.00 0.95"/>
-            </material>
-        </visual>
-        <collision>
-            <origin xyz="0.0 0.0 0.0" rpy="0.0 0.0 0.0"/>
-            <geometry>
-                <mesh filename="${arm_tag_mount_mesh}" scale="1.0 1.0 1.0"/>
-            </geometry>
-        </collision>
-    </link>
-    <joint name="tag_center_offset" type="fixed">
-        <origin xyz="-0.025 0.0 0.04" rpy="0.0 0.0 0.0"/>
-        <parent link="april_tag_mount"/>
-        <child link="tag_center"/>
-    </joint>
-    <link name="tag_center"/>
 </robot>
